File: hardware/v2.5/hat/Planktoscope-Hat.kicad_pcb (KiCad board)
At the start: 2 copper layers, 89.5 x 63.5 mm, 15 parts, among them J1 Conn_01x02_Pin, J2 Conn_01x04_Pin, J3 USB_C_Receptacle_PowerOnly_6P, K1 SSQ-120-04-T-D, Q1 Q_NPN_EBC

Commit message: PCB v2
Parts:
- added J4: FAN, Connector_PinHeader_2.54mm:PinHeader_1x03_P2.54mm_Horizontal, B.Cu at (81.3, 39.2)
- moved J2 5.95 mm to (136.8, 67.7)
- moved R12 0.30 mm to (116.8, 70.5)
- moved J1 0.14 mm to (109.8, 91.8)
Routing:
- net +5V/1: track 70.5 -> 64.2 mm
- net /UART_TX: track 0.00 -> 5.03 mm
- net +12V: track 115.4 -> 114.9 mm
- net GND: vias 2 -> 0
- net (no net): vias 2 -> 4

Commit message: first commint in this repo
Parts:
- removed CTRL1, CTRL2: TMC5160_SILENTSTEPSTICK, mioss:tmc5160 driver
- removed R18, R19: 10k, Diode_SMD:D_1206_3216Metric
- added A4988: ~, mioss:POLOLU_SMD, F.Cu at (143.7, 77.1)
- added A4988_1: ~, mioss:POLOLU_SMD, F.Cu at (141.1, 50.7)
- moved R1 18.2 mm to (106.2, 52.9)
- moved Q1 15.4 mm to (108.7, 60.0), turned to 0 degrees
- moved R7 13.9 mm to (119.6, 67.2), turned to 180 degrees
- moved J2 7.74 mm to (144.3, 65.6)
- moved J1 7.47 mm to (117.2, 91.5)
- moved R12 5.67 mm to (122.4, 69.6), turned to 0 degrees
- moved MOT1-2 5.35 mm to (146.1, 38.7)
- moved LAMP1 4.42 mm to (125.2, 82.2)
- moved MOT2 3.33 mm to (138.7, 91.3)
Connections:
- K1 pad 23: /SPI0_SCLK -> Led
- K1 pad 29: /GPIO5 -> DIR
- K1 pad 31: /GPIO6 -> STEP
- K1 pad 35: /GPIO19 -> STEP_1
- K1 pad 37: /GPIO26 -> DIR_1
- R1 pad 1: /GPIO13/PWM1 -> Led
Routing:
- net /GPIO20: track 84.6 -> 0.00 mm, vias 2 -> 0
- net /GPIO16: track 83.7 -> 0.00 mm, vias 2 -> 0
- net /SPI0_SCLK: track 72.7 -> 0.00 mm, vias 2 -> 0
- net /SPI0_MOSI: track 71.0 -> 0.00 mm, vias 2 -> 0
- net /SPI0_CE0: track 70.6 -> 0.00 mm, vias 2 -> 0
- net /SPI0_CE1: track 66.9 -> 0.00 mm, vias 2 -> 0
- net /SPI0_MISO: track 65.6 -> 0.00 mm
- net /GPIO6: track 59.7 -> 0.00 mm, vias 2 -> 0
- net /GPIO5: track 58.7 -> 0.00 mm
- net STEP_1: track 0.00 -> 42.5 mm
- net DIR_1: track 0.00 -> 39.1 mm
- net DIR: track 0.00 -> 35.7 mm
- net STEP: track 0.00 -> 34.1 mm
- net /GPIO13/PWM1: track 21.0 -> 0.00 mm, vias 3 -> 0
- net Led: track 0.00 -> 7.74 mm
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