File: hardware/v2.5/hat/Planktoscope-Hat.kicad_sch (KiCad schematic)
At the start: 15 parts, among them J1 Conn_01x02_Pin, J2 Conn_01x04_Pin, J3 USB_C_Receptacle_PowerOnly_6P, K1 SSQ-120-04-T-D, Q1 Q_NPN_EBC

Commit message: PCB v2
Parts:
- added J4: FAN, Connector_PinHeader_2.54mm:PinHeader_1x03_P2.54mm_Horizontal, symbol Connector:Conn_01x03_Pin
Connections:
- net +5V/1: now also J4.3 (Pin_3)
- net GND: now also J4.2 (Pin_2)
- net UART_TX: now also J4.1 (Pin_1)
- no-connect marks 0 -> 4

Commit message: first commint in this repo
Parts:
- removed CTRL1, CTRL2: TMC5160_SILENTSTEPSTICK, mioss:tmc5160 driver, symbol Planktoscope-Hat-eagle-import:TMC5160_SILENTSTEPSTICK
- removed R18, R19: 10k, Diode_SMD:D_1206_3216Metric, symbol Planktoscope-Hat-eagle-import:RESISTOR_0805MP
- added A4988, A4988_1: ~, mioss:POLOLU_SMD, symbol oTROSs:polulo_A4988
Connections:
- net SPI0_SCLK is gone; now on net Led: K1.23
- net +12V: now also A4988.9 (Pin_9), A4988_1.9 (Pin_9)
- net +3V3: now also A4988.15 (Pin_15), A4988_1.15 (Pin_15)
- net GND: now also A4988.10 (Pin_10), A4988.16 (Pin_16), A4988_1.10 (Pin_10), A4988_1.16 (Pin_16)
- net at MOT2.1: now also A4988.14 (Pin_14)
- net at MOT2.2: now also A4988.13 (Pin_13)
- net at MOT2.3: now also A4988.12 (Pin_12)
- net at MOT2.4: now also A4988.11 (Pin_11)
- net at MOT1-2.1: now also A4988_1.14 (Pin_14)
- net at MOT1-2.2: now also A4988_1.13 (Pin_13)
- net at MOT1-2.3: now also A4988_1.12 (Pin_12)
- net at MOT1-2.4: now also A4988_1.11 (Pin_11)
- net GPIO13/PWM1 renamed Led
- net GPIO19 renamed STEP_1
- net STEP_1: now also A4988_1.7 (Pin_7)
- net GPIO26 renamed DIR_1
- net DIR_1: now also A4988_1.8 (Pin_8)
- net GPIO5 renamed DIR
- net DIR: now also A4988.8 (Pin_8)
- net GPIO6 renamed STEP
- net STEP: now also A4988.7 (Pin_7)
- new net: A4988.5 (Pin_5), A4988.6 (Pin_6)
- new net: A4988_1.5 (Pin_5), A4988_1.6 (Pin_6)
- no-connect marks 4 -> 0
Other:
- note removed: "Pull-up for DRV_EN"
- moved on the sheet: MOT1-2, MOT2
